Commit message: Update sick_m8.urdf.xacro

File: husky_description/urdf/accessories/sick_m8.urdf.xacro (robot description, xacro)
@@ -2,11 +2,6 @@
 <robot xmlns:xacro="http://www.ros.org/wiki/xacro" name="VLP-16">
   <xacro:property name="M_PI" value="3.1415926535897931" />
-  <xacro:macro name="VLP-16" params="*origin namespace parent:=base_link name:=M8 topic:=M8_points hz:=10 lasers:=8 samples:=1875 collision_range:=0.3 min_range:=0.9 max_range:=200.0 noise:=0.008 min_angle:=-${M_PI} max_angle:=${M_PI}">
-    <joint name="${namespace}/${name}_base_mount_joint" type="fixed">
-      <xacro:insert_block name="origin" />
-      <parent link="${namespace}/${parent}"/>
-      <child link="${namespace}/${name}_base_link"/>
-    </joint>
-    <link name="${namespace}/${name}_base_link">
+  <xacro:macro name="sick_m8" params="*origin namespace parent:=base_link name:=m8_husky topic:=/m8_husky_lidar hz:=10 lasers:=8 samples:=1875 collision_range:=0.3 min_range:=0.9 max_range:=200.0 noise:=0.008 min_angle:=-${M_PI} max_angle:=${M_PI}">
+    <link name="${frame}">
       <inertial>
         <mass value="0.564"/>
@@ -28,32 +23,15 @@
       </collision>
     </link>
-    <joint name="${namespace}/${name}_base_scan_joint" type="fixed" >
-      <origin xyz="0 0 0.0377" rpy="0 0 0" />
-      <parent link="${namespace}/${name}_base_link" />
-      <child link="${namespace}/${name}"/>
-    </joint>
-    <link name="${namespace}/${name}">
-      <inertial>
-        <mass value="0.564"/>
-        <origin xyz="0 0 0"/>
-        <inertia ixx="0.003881243" ixy="0" ixz="0" iyy="0.000498940" iyz="0" izz="0.003879257"/>
-      </inertial>
-      <visual>
-        <origin xyz="0 0 -0.0377" />
-        <geometry>
-          <mesh filename="package://velodyne_description/meshes/M8.dae" />
-        </geometry>
-      </visual>
-    </link>
     <!-- Gazebo requires the velodyne_gazebo_plugins package -->
-    <gazebo reference="${namespace}/${name}">
-      <sensor type="ray" name="${namespace}/${name}-VLP16">
+     <gazebo reference="${frame}">
+      <turnGravityOff>true</turnGravityOff>
+      <sensor type="ray" name="${frame}">
         <pose>0 0 0 0 0 0</pose>
         <visualize>false</visualize>
-        <update_rate>${hz}</update_rate>
+        <update_rate>${update_rate}</update_rate>
         <ray>
           <scan>
             <horizontal>
-              <samples>${samples}</samples>
+              <samples>${sample_size}</samples>
               <resolution>1</resolution>
               <min_angle>${min_angle}</min_angle>
@@ -61,24 +39,24 @@
             </horizontal>
             <vertical>
-              <samples>${lasers}</samples>
+              <samples>8</samples>
               <resolution>1</resolution>
-              <min_angle>-${17.0*M_PI/180.0}</min_angle>
-              <max_angle> ${3.0*M_PI/180.0}</max_angle>
+              <min_angle>-${3.0*M_PI/180.0}</min_angle>
+              <max_angle> ${17.0*M_PI/180.0}</max_angle>
             </vertical>
           </scan>
           <range>
-            <min>${collision_range}</min>
-            <max>${max_range+1}</max>
-            <resolution>0.001</resolution>
+            <min>${min_range}</min>
+            <max>${max_range}</max>
+            <resolution>0.01</resolution>
           </range>
           <noise>
             <type>gaussian</type>
             <mean>0.0</mean>
-            <stddev>0.2</stddev>
+            <stddev>0.001</stddev>
           </noise>
         </ray>
         <plugin name="gazebo_ros_laser_controller" filename="libgazebo_ros_velodyne_laser.so">
           <topicName>${topic}</topicName>
-          <frameName>/${namespace}/${name}</frameName>
+          <frameName>${frame}</frameName>
           <min_range>${min_range}</min_range>
           <max_range>${max_range}</max_range>
