Commit message: Update husky_tf.urdf.xacro

File: husky_description/urdf/husky_tf.urdf.xacro (robot description, xacro)
@@ -9,7 +9,8 @@
 -->
 <robot name="husky" xmlns:xacro="http://ros.org/wiki/xacro">
+  <xacro:property name="M_PI" value="3.1415926535897931" />
   <xacro:arg name="laser_enabled" default="false" />
-  <xacro:arg name="laser_xyz" default="$(optenv HUSKY_LMS1XX_XYZ 0.2206 0.0 0.00635)" />
-  <xacro:arg name="laser_rpy" default="$(optenv HUSKY_LMS1XX_RPY 0.0 0.0 0.0)" />
+  <xacro:arg name="laser_xyz" default="$(optenv HUSKY_LMS1XX_XYZ 0.35 0.0 0.006)" />
+  <xacro:arg name="laser_rpy" default="$(optenv HUSKY_LMS1XX_RPY 0.0 -${M_PI/360*300} 0.0)" />
   <xacro:arg name="kinect_enabled" default="false" />
   <xacro:arg name="kinect_xyz" default="$(optenv HUSKY_KINECT_XYZ 0 0 0)" />
@@ -22,5 +23,5 @@
   <xacro:include filename="$(find husky_description)/urdf/wheel_tf.urdf.xacro" />
   <xacro:include filename="$(find husky_description)/urdf/accessories/kinect_camera.urdf.xacro"/>
-  <xacro:include filename="$(find husky_description)/urdf/accessories/sick_lms1xx_mount.urdf.xacro"/>
+  <xacro:include filename="$(find husky_description)/urdf/accessories/sick_m8_mount.urdf.xacro"/>
   <xacro:include filename="$(find husky_description)/urdf/accessories/sensor_arch.urdf.xacro"/>
   <xacro:property name="M_PI" value="3.14159"/>
@@ -102,6 +103,6 @@
   <xacro:husky_decorate tf_prefix="$(arg tf_prefix)"/>
   <xacro:if value="$(arg laser_enabled)">
-    <sick_lms1xx_mount prefix="$(arg tf_prefix)/base"/>
-    <sick_lms1xx frame="$(arg tf_prefix)/base_laser" topic="scan"/>
+    <sick_m8_mount prefix="$(arg tf_prefix)/base"/>
+    <sick_m8 frame="$(arg tf_prefix)/base_laser" topic="scan"/>
     <joint name="$(arg tf_prefix)/laser_mount_joint" type="fixed">
       <origin xyz="$(arg laser_xyz)" rpy="$(arg laser_rpy)" />

Commit message: Update husky_tf.urdf.xacro

File: husky_description/urdf/husky_tf.urdf.xacro (robot description, xacro)
@@ -25,5 +25,4 @@
   <xacro:include filename="$(find husky_description)/urdf/accessories/sick_m8_mount.urdf.xacro"/>
   <xacro:include filename="$(find husky_description)/urdf/accessories/sensor_arch.urdf.xacro"/>
-  <xacro:property name="M_PI" value="3.14159"/>
   <!-- Base Size -->
   <xacro:property name="base_x_size" value="0.98740000" />
@@ -104,5 +103,5 @@
   <xacro:if value="$(arg laser_enabled)">
     <sick_m8_mount prefix="$(arg tf_prefix)/base"/>
-    <sick_m8 frame="$(arg tf_prefix)/base_laser" topic="scan"/>
+    <sick_m8 frame="$(arg tf_prefix)/base_laser" topic="m8_husky_lidar" robot_namespace="$(arg robot_namespace)"/>
     <joint name="$(arg tf_prefix)/laser_mount_joint" type="fixed">
       <origin xyz="$(arg laser_xyz)" rpy="$(arg laser_rpy)" />
